File: MPF-III/Keyboard/MPF-III_Keyboard/MPF-III_Keyboard.kicad_sch (KiCad schematic)
At the start: 2 parts, among them J1 MPF-III U78, J2 MPF-III Keyboard Socket

Commit message: Started schematic design
Parts:
- added D1: CAPS LOCK, LED_THT:LED_D5.0mm, symbol Device:LED
- added D2: NUM LOCK, LED_THT:LED_D5.0mm, symbol Device:LED
- added R1, R2: R, Resistor_THT:R_Axial_DIN0207_L6.3mm_D2.5mm_P10.16mm_Horizontal, symbol Device:R
- added SW1: F1, PCM_Switch_Keyboard_Cherry_MX:SW_Cherry_MX_PCB_1.00u, symbol Switch:SW_Push_45deg
- added SW10: F10, PCM_Switch_Keyboard_Cherry_MX:SW_Cherry_MX_PCB_1.00u, symbol Switch:SW_Push_45deg
- added SW11: F11, PCM_Switch_Keyboard_Cherry_MX:SW_Cherry_MX_PCB_1.00u, symbol Switch:SW_Push_45deg
- added SW12: F12, PCM_Switch_Keyboard_Cherry_MX:SW_Cherry_MX_PCB_1.00u, symbol Switch:SW_Push_45deg
- added SW13: PB0, PCM_Switch_Keyboard_Cherry_MX:SW_Cherry_MX_PCB_1.00u, symbol Switch:SW_Push_45deg
- added SW14: PB1, PCM_Switch_Keyboard_Cherry_MX:SW_Cherry_MX_PCB_1.00u, symbol Switch:SW_Push_45deg
- added SW15: BREAK, PCM_Switch_Keyboard_Cherry_MX:SW_Cherry_MX_PCB_1.00u, symbol Switch:SW_Push_45deg
- added SW16: RESET, PCM_Switch_Keyboard_Cherry_MX:SW_Cherry_MX_PCB_1.00u, symbol Switch:SW_Push_45deg
- added SW17: NUM LOCK, PCM_Switch_Keyboard_Cherry_MX:SW_Cherry_MX_PCB_2.00u, symbol Switch:SW_Push_45deg
- added SW18: HALT, PCM_Switch_Keyboard_Cherry_MX:SW_Cherry_MX_PCB_2.00u, symbol Switch:SW_Push_45deg
- added SW19: ESC, PCM_Switch_Keyboard_Cherry_MX:SW_Cherry_MX_PCB_1.00u, symbol Switch:SW_Push_45deg
- added SW2: F2, PCM_Switch_Keyboard_Cherry_MX:SW_Cherry_MX_PCB_1.00u, symbol Switch:SW_Push_45deg
- added SW20: ! 1, PCM_Switch_Keyboard_Cherry_MX:SW_Cherry_MX_PCB_1.00u, symbol Switch:SW_Push_45deg
- added SW21: @ 2, PCM_Switch_Keyboard_Cherry_MX:SW_Cherry_MX_PCB_1.00u, symbol Switch:SW_Push_45deg
- added SW22: # 3, PCM_Switch_Keyboard_Cherry_MX:SW_Cherry_MX_PCB_1.00u, symbol Switch:SW_Push_45deg
- added SW23: $ 4, PCM_Switch_Keyboard_Cherry_MX:SW_Cherry_MX_PCB_1.00u, symbol Switch:SW_Push_45deg
- added SW24: % 5, PCM_Switch_Keyboard_Cherry_MX:SW_Cherry_MX_PCB_1.00u, symbol Switch:SW_Push_45deg
- added SW25: ^ 6, PCM_Switch_Keyboard_Cherry_MX:SW_Cherry_MX_PCB_1.00u, symbol Switch:SW_Push_45deg
- added SW26: & 7, PCM_Switch_Keyboard_Cherry_MX:SW_Cherry_MX_PCB_1.00u, symbol Switch:SW_Push_45deg
- added SW27: * 8, PCM_Switch_Keyboard_Cherry_MX:SW_Cherry_MX_PCB_1.00u, symbol Switch:SW_Push_45deg
- added SW28: ( 9, PCM_Switch_Keyboard_Cherry_MX:SW_Cherry_MX_PCB_1.00u, symbol Switch:SW_Push_45deg
- added SW29: ) 0, PCM_Switch_Keyboard_Cherry_MX:SW_Cherry_MX_PCB_1.00u, symbol Switch:SW_Push_45deg
- added SW3: F3, PCM_Switch_Keyboard_Cherry_MX:SW_Cherry_MX_PCB_1.00u, symbol Switch:SW_Push_45deg
- added SW30: _ -, PCM_Switch_Keyboard_Cherry_MX:SW_Cherry_MX_PCB_1.00u, symbol Switch:SW_Push_45deg
- added SW31: + =, PCM_Switch_Keyboard_Cherry_MX:SW_Cherry_MX_PCB_1.00u, symbol Switch:SW_Push_45deg
- added SW32: <--, PCM_Switch_Keyboard_Cherry_MX:SW_Cherry_MX_PCB_2.00u, symbol Switch:SW_Push_45deg
- added SW33: TAB, PCM_Switch_Keyboard_Cherry_MX:SW_Cherry_MX_PCB_1.50u, symbol Switch:SW_Push_45deg
- added SW34: Q, PCM_Switch_Keyboard_Cherry_MX:SW_Cherry_MX_PCB_1.00u, symbol Switch:SW_Push_45deg
- added SW35: W, PCM_Switch_Keyboard_Cherry_MX:SW_Cherry_MX_PCB_1.00u, symbol Switch:SW_Push_45deg
- added SW36: E, PCM_Switch_Keyboard_Cherry_MX:SW_Cherry_MX_PCB_1.00u, symbol Switch:SW_Push_45deg
- added SW37: R, PCM_Switch_Keyboard_Cherry_MX:SW_Cherry_MX_PCB_1.00u, symbol Switch:SW_Push_45deg
- added SW38: T, PCM_Switch_Keyboard_Cherry_MX:SW_Cherry_MX_PCB_1.00u, symbol Switch:SW_Push_45deg
- added SW39: Y, PCM_Switch_Keyboard_Cherry_MX:SW_Cherry_MX_PCB_1.00u, symbol Switch:SW_Push_45deg
- added SW4: F4, PCM_Switch_Keyboard_Cherry_MX:SW_Cherry_MX_PCB_1.00u, symbol Switch:SW_Push_45deg
- added SW40: U, PCM_Switch_Keyboard_Cherry_MX:SW_Cherry_MX_PCB_1.00u, symbol Switch:SW_Push_45deg
- added SW41: I, PCM_Switch_Keyboard_Cherry_MX:SW_Cherry_MX_PCB_1.00u, symbol Switch:SW_Push_45deg
- added SW42: O, PCM_Switch_Keyboard_Cherry_MX:SW_Cherry_MX_PCB_1.00u, symbol Switch:SW_Push_45deg
- added SW43: P, PCM_Switch_Keyboard_Cherry_MX:SW_Cherry_MX_PCB_1.00u, symbol Switch:SW_Push_45deg
- added SW44: { [, PCM_Switch_Keyboard_Cherry_MX:SW_Cherry_MX_PCB_1.00u, symbol Switch:SW_Push_45deg
- added SW45: } ], PCM_Switch_Keyboard_Cherry_MX:SW_Cherry_MX_PCB_1.00u, symbol Switch:SW_Push_45deg
- added SW46: DEL, PCM_Switch_Keyboard_Cherry_MX:SW_Cherry_MX_PCB_1.50u, symbol Switch:SW_Push_45deg
- added SW47: NP 7, PCM_Switch_Keyboard_Cherry_MX:SW_Cherry_MX_PCB_1.00u, symbol Switch:SW_Push_45deg
- added SW48: NP 8, PCM_Switch_Keyboard_Cherry_MX:SW_Cherry_MX_PCB_1.00u, symbol Switch:SW_Push_45deg
- added SW49: NP 9, PCM_Switch_Keyboard_Cherry_MX:SW_Cherry_MX_PCB_1.00u, symbol Switch:SW_Push_45deg
- added SW5: F5, PCM_Switch_Keyboard_Cherry_MX:SW_Cherry_MX_PCB_1.00u, symbol Switch:SW_Push_45deg
- added SW50: NP -, PCM_Switch_Keyboard_Cherry_MX:SW_Cherry_MX_PCB_1.00u, symbol Switch:SW_Push_45deg
- added SW51: NP 4, PCM_Switch_Keyboard_Cherry_MX:SW_Cherry_MX_PCB_1.00u, symbol Switch:SW_Push_45deg
- added SW52: NP 5, PCM_Switch_Keyboard_Cherry_MX:SW_Cherry_MX_PCB_1.00u, symbol Switch:SW_Push_45deg
- added SW53: NP 6, PCM_Switch_Keyboard_Cherry_MX:SW_Cherry_MX_PCB_1.00u, symbol Switch:SW_Push_45deg
- added SW54: NP +, PCM_Switch_Keyboard_Cherry_MX:SW_Cherry_MX_PCB_1.00u, symbol Switch:SW_Push_45deg
- added SW55: CTRL, PCM_Switch_Keyboard_Cherry_MX:SW_Cherry_MX_PCB_2.00u, symbol Switch:SW_Push_45deg
- added SW56: A, PCM_Switch_Keyboard_Cherry_MX:SW_Cherry_MX_PCB_1.00u, symbol Switch:SW_Push_45deg
- added SW57: S, PCM_Switch_Keyboard_Cherry_MX:SW_Cherry_MX_PCB_1.00u, symbol Switch:SW_Push_45deg
- added SW58: D, PCM_Switch_Keyboard_Cherry_MX:SW_Cherry_MX_PCB_1.00u, symbol Switch:SW_Push_45deg
- added SW59: F, PCM_Switch_Keyboard_Cherry_MX:SW_Cherry_MX_PCB_1.00u, symbol Switch:SW_Push_45deg
- added SW6: F6, PCM_Switch_Keyboard_Cherry_MX:SW_Cherry_MX_PCB_1.00u, symbol Switch:SW_Push_45deg
- added SW60: G, PCM_Switch_Keyboard_Cherry_MX:SW_Cherry_MX_PCB_1.00u, symbol Switch:SW_Push_45deg
- added SW61: H, PCM_Switch_Keyboard_Cherry_MX:SW_Cherry_MX_PCB_1.00u, symbol Switch:SW_Push_45deg
- added SW62: J, PCM_Switch_Keyboard_Cherry_MX:SW_Cherry_MX_PCB_1.00u, symbol Switch:SW_Push_45deg
- added SW63: K, PCM_Switch_Keyboard_Cherry_MX:SW_Cherry_MX_PCB_1.00u, symbol Switch:SW_Push_45deg
- added SW64: L, PCM_Switch_Keyboard_Cherry_MX:SW_Cherry_MX_PCB_1.00u, symbol Switch:SW_Push_45deg
- added SW65: : ;, PCM_Switch_Keyboard_Cherry_MX:SW_Cherry_MX_PCB_1.00u, symbol Switch:SW_Push_45deg
- added SW66: " ', PCM_Switch_Keyboard_Cherry_MX:SW_Cherry_MX_PCB_1.00u, symbol Switch:SW_Push_45deg
- added SW67: ~ `, PCM_Switch_Keyboard_Cherry_MX:SW_Cherry_MX_PCB_1.00u, symbol Switch:SW_Push_45deg
- added SW68: RETURN, PCM_Switch_Keyboard_Cherry_MX:SW_Cherry_MX_PCB_2.00u_90deg, symbol Switch:SW_Push_45deg
- added SW69: NP 1, PCM_Switch_Keyboard_Cherry_MX:SW_Cherry_MX_PCB_1.00u, symbol Switch:SW_Push_45deg
- added SW7: F7, PCM_Switch_Keyboard_Cherry_MX:SW_Cherry_MX_PCB_1.00u, symbol Switch:SW_Push_45deg
- added SW70: NP 2, PCM_Switch_Keyboard_Cherry_MX:SW_Cherry_MX_PCB_1.00u, symbol Switch:SW_Push_45deg
- added SW71: NP 3, PCM_Switch_Keyboard_Cherry_MX:SW_Cherry_MX_PCB_1.00u, symbol Switch:SW_Push_45deg
- added SW72: NP RETURN, PCM_Switch_Keyboard_Cherry_MX:SW_Cherry_MX_PCB_2.00u_90deg, symbol Switch:SW_Push_45deg
- added SW73: LH SHIFT, PCM_Switch_Keyboard_Cherry_MX:SW_Cherry_MX_PCB_1.50u, symbol Switch:SW_Push_45deg
- added SW74: | \, PCM_Switch_Keyboard_Cherry_MX:SW_Cherry_MX_PCB_1.00u, symbol Switch:SW_Push_45deg
- added SW75: Z, PCM_Switch_Keyboard_Cherry_MX:SW_Cherry_MX_PCB_1.00u, symbol Switch:SW_Push_45deg
- added SW76: X, PCM_Switch_Keyboard_Cherry_MX:SW_Cherry_MX_PCB_1.00u, symbol Switch:SW_Push_45deg
- added SW77: C, PCM_Switch_Keyboard_Cherry_MX:SW_Cherry_MX_PCB_1.00u, symbol Switch:SW_Push_45deg
- added SW78: V, PCM_Switch_Keyboard_Cherry_MX:SW_Cherry_MX_PCB_1.00u, symbol Switch:SW_Push_45deg
- added SW79: B, PCM_Switch_Keyboard_Cherry_MX:SW_Cherry_MX_PCB_1.00u, symbol Switch:SW_Push_45deg
- added SW8: F8, PCM_Switch_Keyboard_Cherry_MX:SW_Cherry_MX_PCB_1.00u, symbol Switch:SW_Push_45deg
- added SW80: N, PCM_Switch_Keyboard_Cherry_MX:SW_Cherry_MX_PCB_1.00u, symbol Switch:SW_Push_45deg
- added SW81: M, PCM_Switch_Keyboard_Cherry_MX:SW_Cherry_MX_PCB_1.00u, symbol Switch:SW_Push_45deg
- added SW82: < ,, PCM_Switch_Keyboard_Cherry_MX:SW_Cherry_MX_PCB_1.00u, symbol Switch:SW_Push_45deg
- added SW83: > ., PCM_Switch_Keyboard_Cherry_MX:SW_Cherry_MX_PCB_1.00u, symbol Switch:SW_Push_45deg
- added SW84: ? /, PCM_Switch_Keyboard_Cherry_MX:SW_Cherry_MX_PCB_1.00u, symbol Switch:SW_Push_45deg
- added SW85: RH SHIFT, PCM_Switch_Keyboard_Cherry_MX:SW_Cherry_MX_PCB_1.50u, symbol Switch:SW_Push_45deg
- added SW86: ALT, PCM_Switch_Keyboard_Cherry_MX:SW_Cherry_MX_PCB_2.25u, symbol Switch:SW_Push_45deg
- added SW87: SPACE, PCM_Switch_Keyboard_Cherry_MX:SW_Cherry_MX_PCB_7.00u, symbol Switch:SW_Push_45deg
- added SW88: CAPS LOCK, PCM_Switch_Keyboard_Cherry_MX:SW_Cherry_MX_PCB_2.00u, symbol Switch:SW_Push_45deg
- added SW89: NP 0, PCM_Switch_Keyboard_Cherry_MX:SW_Cherry_MX_PCB_2.00u, symbol Switch:SW_Push_45deg
- added SW9: F9, PCM_Switch_Keyboard_Cherry_MX:SW_Cherry_MX_PCB_1.00u, symbol Switch:SW_Push_45deg
- added SW90: NP dot, PCM_Switch_Keyboard_Cherry_MX:SW_Cherry_MX_PCB_2.00u, symbol Switch:SW_Push_45deg
- J2: footprint (none) -> Connector_Dsub:DSUB-9_Pins_Horizontal_P2.77x2.84mm_EdgePinOffset7.70mm_Housed_MountingHolesOffset9.12mm
Connections:
- net GND: now also D1.1 (K), D2.1 (K)
- new net: D1.2 (A), R1.1
- new net: D2.2 (A), R2.1
Other:
- note added: "WAITING FOR CONFIRMATION OF THE KEYBOARD MATRIX"
- company: (none) -> Brett Hallen
- title: (none) -> Multitech Micro Professor MPF-III Keyboard
- moved on the sheet: J1, J2
